File: hardware/backplane/SENTINEL_BACKPLANE.kicad_pcb (KiCad board)
At the start: 4 copper layers, 232 x 112 mm, 57 parts, among them J1 SLOT1, J10 50V IN, J11 DRAIN1, J12 DRAIN2, J13 DRAIN3, J14 DRAIN4, J15 DRAIN5, J16 DRAIN6, J17 DRAIN7, J18 DRAIN8, J19 12V IN, J2 SLOT2, J3 SLOT3, J4 SLOT4, J5 SLOT5, J6 SLOT6, J7 SLOT7, J8 SLOT8, J9 TO TILE

Commit message: Five boards DRC-clean, BOMs, layout engine improvements
- Backplane, clock & timing, calibration network, PSU and feed board layouts now pass
  KiCad DRC with zero errors and zero unconnected items
- T/R module: 0 DRC errors, 6 connections left to route by hand
- Calibration selector redesigned as an SPDT tree (replaces the fine-pitch SP8T)
- PSU: IPC-2221 2.5 mm high-voltage clearance via KiCad custom rules
- Backplane/tile cable re-pinned (slots 1-4 left column, 5-8 right) for routability
- Grouped BOM CSV for every board (hardware/tools/export_bom.sh)
- Router: partial routing, neck-downs at fine-pitch pins, long-axis fan-out,
  NPTH obstacles, pour-net connectivity, domain-aware clearance, rip-up tuning

Co-Authored-By: Claude Opus 5.5 <noreply@anthropic.com>
Parts:
- moved J9 40.7 mm to (114.0, 60.5), turned to 0 degrees
- moved R5 20.5 mm to (120.5, 100.8)
- moved R6 20.5 mm to (124.9, 100.8)
- moved R7 20.4 mm to (129.3, 100.8)
- moved R8 20.4 mm to (133.7, 100.8)
- moved R4 20.2 mm to (108.7, 100.8)
- moved R3 20.1 mm to (104.3, 100.8)
- moved R2 20.1 mm to (99.9, 100.8)
- moved R1 20.1 mm to (95.5, 100.8)
Connections:
- J9 pad 10: TX_EN_T3 -> RS485_A6
- J9 pad 11: RS485_B3 -> RS485_B2
- J9 pad 12: FAULT_N3 -> RS485_B6
- J9 pad 13: RS485_A4 -> TX_EN_T2
- J9 pad 14: TX_EN_T4 -> TX_EN_T6
- J9 pad 15: RS485_B4 -> FAULT_N2
- J9 pad 16: FAULT_N4 -> FAULT_N6
- J9 pad 17: RS485_A5 -> RS485_A3
- J9 pad 18: TX_EN_T5 -> RS485_A7
- J9 pad 19: RS485_B5 -> RS485_B3
- J9 pad 2: TX_EN_T1 -> RS485_A5
- J9 pad 20: FAULT_N5 -> RS485_B7
- J9 pad 21: RS485_A6 -> TX_EN_T3
- J9 pad 22: TX_EN_T6 -> TX_EN_T7
- J9 pad 23: RS485_B6 -> FAULT_N3
- J9 pad 24: FAULT_N6 -> FAULT_N7
- J9 pad 25: RS485_A7 -> RS485_A4
- J9 pad 26: TX_EN_T7 -> RS485_A8
- J9 pad 27: RS485_B7 -> RS485_B4
- J9 pad 28: FAULT_N7 -> RS485_B8
- J9 pad 29: RS485_A8 -> TX_EN_T4
- J9 pad 31: RS485_B8 -> FAULT_N4
- J9 pad 4: FAULT_N1 -> RS485_B5
- J9 pad 5: RS485_A2 -> TX_EN_T1
- J9 pad 6: TX_EN_T2 -> TX_EN_T5
- J9 pad 7: RS485_B2 -> FAULT_N1
- J9 pad 8: FAULT_N2 -> FAULT_N5
- J9 pad 9: RS485_A3 -> RS485_A2
Routing:
- net RS485_A1: track 0.00 -> 133.4 mm, vias 0 -> 2
- net RS485_B1: track 0.00 -> 129.1 mm, vias 0 -> 1
- net RS485_B2: track 0.00 -> 101.5 mm, vias 0 -> 1
- net RS485_A2: track 0.00 -> 101.2 mm
- net RS485_A3: track 0.00 -> 84.9 mm, vias 0 -> 2
- net RS485_B3: track 0.00 -> 84.8 mm, vias 0 -> 3
- net VDD_50V: track 5.95 -> 74.4 mm
- net RS485_B5: track 113.2 -> 47.8 mm, vias 1 -> 0
- net RS485_A5: track 110.5 -> 47.8 mm, vias 1 -> 0
- net RS485_A6: track 123.0 -> 70.8 mm
- net RS485_B6: track 114.0 -> 72.1 mm, vias 2 -> 1
- net FAULT_N8: track 96.2 -> 131.7 mm, vias 1 -> 3
- net FAULT_N5: track 79.9 -> 47.9 mm
- net TX_EN_T4: track 38.4 -> 8.77 mm, vias 2 -> 1
- net RS485_B4: track 112.2 -> 83.8 mm, vias 2 -> 3
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