File: hardware/rfsoc_tile/SENTINEL_TILE.kicad_pcb (KiCad board)
At the start: 4 copper layers, 240 x 190 mm, 118 parts, among them J1 SOM CONN A, J10 RX1, J11 RX2, J12 RX3, J13 RX4, J14 RX5, J15 RX6, J16 RX7, J17 RX8, J18 RXCAL, J2 SOM CONN B, J20 TX1, J21 TX2, J22 TX3, J23 TX4, J24 TX5, J25 TX6, J26 TX7, J27 TX8, J28 TXCAL, J3 BACKPLANE, J4 CLOCK, J5 CAL CTRL, J6 PSU LINK, J7 QSFP28, J8 12V IN, T1 1:2, T11 1:2, T12 1:2, T13 1:2, T14 1:2, T15 1:2, T16 1:2, T17 1:2, T18 1:2, T19 1:2, T2 1:2, T3 1:2, T4 1:2, T5 1:2, T6 1:2, T7 1:2, T8 1:2, T9 1:2, U1 THVD1450, U10 LMR33630, U2 THVD1450, U3 THVD1450, U4 THVD1450, U5 THVD1450, U6 THVD1450, U7 THVD1450, U8 THVD1450, U9 THVD1450

Commit message: RFSoC tile: 320 x 260 mm, routed with EasyEDA Pro, DRC clean
- Board enlarged from 240 x 190 to 320 x 260 mm; SOM connector B pins
  grouped by row toward their destinations (RS-485 / control side).
- Routing done by the EasyEDA Pro autorouter (Top / In2 / Bottom, In1 kept
  as solid GND) and imported back into KiCad: 0 DRC errors, 0 unrouted.
- tools/import_easyeda.py replays easyeda_routes.json onto the KiCad board;
  tools/layer_preview.py draws copper previews from any finished board.
- Regenerated gerbers, 3D view, BOM, figures, report and README (6 of 7
  layouts now DRC clean).

Co-Authored-By: Claude Opus 5.5 <noreply@anthropic.com>
Parts:
- moved C25 131.6 mm to (267.5, 229.6)
- moved C8 128.3 mm to (264.8, 186.8)
- moved R22 121.8 mm to (277.9, 28.8)
- moved R21 120.8 mm to (271.9, 28.8)
- moved J28 105.0 mm to (317.1, 234.0)
- moved T19 105.0 mm to (305.0, 234.0)
- moved J27 100.0 mm to (317.1, 207.0)
- moved T18 100.0 mm to (305.0, 207.0)
- moved J26 95.4 mm to (317.1, 180.0)
- moved T17 95.4 mm to (305.0, 180.0)
- moved H3 92.6 mm to (288.0, 170.0)
- moved J25 91.3 mm to (317.1, 153.0)
- moved T16 91.3 mm to (305.0, 153.0)
- moved R27 88.6 mm to (261.3, 228.8)
- moved C24 88.1 mm to (255.0, 229.6)
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Connections:
- J2 pad 1: TXD1 -> PPS_P
- J2 pad 10: FAULT_N2 -> FAULT_N1
- J2 pad 11: TXD3 -> CAL_SW_EN
- J2 pad 12: RXD3 -> TXD2
- J2 pad 13: DE3 -> CAL_INJ_MEAS
- J2 pad 14: TX_EN_T3 -> RXD2
- J2 pad 15: FAULT_N3 -> PSU_TXD
- J2 pad 16: TXD4 -> DE2
- J2 pad 17: RXD4 -> PSU_RXD
- J2 pad 18: DE4 -> TX_EN_T2
- J2 pad 19: TX_EN_T4 -> PSU_DE
- J2 pad 2: RXD1 -> TXD1
- J2 pad 20: FAULT_N4 -> FAULT_N2
- J2 pad 21: TXD5 -> MGT_REFCLK_P
- J2 pad 22: RXD5 -> TXD3
- J2 pad 23: DE5 -> MGT_REFCLK_N
- J2 pad 24: TX_EN_T5 -> RXD3
- J2 pad 25: FAULT_N5 -> QSFP_SCL
- J2 pad 26: TXD6 -> DE3
- J2 pad 27: RXD6 -> QSFP_SDA
- J2 pad 28: DE6 -> TX_EN_T3
- J2 pad 29: TX_EN_T6 -> QSFP_MODSEL
- J2 pad 3: DE1 -> PPS_N
- J2 pad 30: FAULT_N6 -> FAULT_N3
- J2 pad 31: TXD7 -> QSFP_RESET
- J2 pad 32: RXD7 -> TXD4
- J2 pad 33: DE7 -> QSFP_LPMODE
- J2 pad 34: TX_EN_T7 -> RXD4
- J2 pad 35: FAULT_N7 -> QSFP_INT
- J2 pad 36: TXD8 -> DE4
- J2 pad 37: RXD8 -> QSFP_PRS
- J2 pad 38: DE8 -> TX_EN_T4
- J2 pad 39: TX_EN_T8 -> QTX0_P
- J2 pad 4: TX_EN_T1 -> RXD1
- J2 pad 40: FAULT_N8 -> FAULT_N4
- J2 pad 41: CAL_SEL0 -> QTX0_N
- J2 pad 42: CAL_SEL1 -> TXD5
- J2 pad 43: CAL_SEL2 -> QRX0_P
- J2 pad 44: CAL_SW_EN -> RXD5
- J2 pad 45: CAL_INJ_MEAS -> QRX0_N
- J2 pad 46: PPS_P -> DE5
- J2 pad 47: PPS_N -> QTX1_P
- J2 pad 48: PSU_TXD -> TX_EN_T5
- J2 pad 49: PSU_RXD -> QTX1_N
- J2 pad 5: FAULT_N1 -> CAL_SEL0
- J2 pad 50: PSU_DE -> FAULT_N5
- J2 pad 51: QSFP_SCL -> QRX1_P
- J2 pad 52: QSFP_SDA -> TXD6
- J2 pad 53: QSFP_MODSEL -> QRX1_N
- J2 pad 54: QSFP_RESET -> RXD6
- J2 pad 55: QSFP_LPMODE -> QTX2_P
- J2 pad 56: QSFP_INT -> DE6
- J2 pad 57: QSFP_PRS -> QTX2_N
- J2 pad 58: MGT_REFCLK_P -> TX_EN_T6
- J2 pad 59: MGT_REFCLK_N -> QRX2_P
- J2 pad 6: TXD2 -> DE1
- J2 pad 60: QTX0_P -> FAULT_N6
- J2 pad 61: QTX0_N -> QRX2_N
- J2 pad 62: QRX0_P -> TXD7
- J2 pad 63: QRX0_N -> QTX3_P
- J2 pad 64: QTX1_P -> RXD7
- J2 pad 65: QTX1_N -> QTX3_N
- J2 pad 66: QRX1_P -> DE7
- J2 pad 67: QRX1_N -> QRX3_P
- J2 pad 68: QTX2_P -> TX_EN_T7
- J2 pad 69: QTX2_N -> QRX3_N
- J2 pad 7: RXD2 -> CAL_SEL1
- J2 pad 70: QRX2_P -> FAULT_N7
- J2 pad 71: QRX2_N -> +12V
- J2 pad 72: QTX3_P -> TXD8
- J2 pad 73: QTX3_N -> +12V
- J2 pad 74: QRX3_P -> RXD8
- J2 pad 75: QRX3_N -> +12V
- J2 pad 76: +12V -> DE8
- J2 pad 78: +12V -> TX_EN_T8
- J2 pad 8: DE2 -> TX_EN_T1
- J2 pad 80: +12V -> FAULT_N8
- J2 pad 82: +12V -> GND
- J2 pad 83: GND -> +12V
- J2 pad 9: TX_EN_T2 -> CAL_SEL2
Routing:
- net GND: track 192.0 -> 1884.0 mm, vias 2001 -> 47
- net DAC8_N: track 2.75 -> 227.5 mm
- net QSFP_INT: track 40.5 -> 260.7 mm, vias 4 -> 3
- net DAC7_N: track 2.75 -> 211.7 mm
- net ADC8_P: track 2.73 -> 210.3 mm
- net QSFP_MODSEL: track 3.40 -> 203.9 mm, vias 2 -> 4
- net QRX1_N: track 3.15 -> 202.3 mm, vias 2 -> 3
- net DAC6_N: track 2.75 -> 201.3 mm
- net QRX1_P: track 4.65 -> 201.7 mm, vias 2 -> 3
- net QSFP_RESET: track 2.90 -> 198.5 mm, vias 2 -> 3
- net QTX3_N: track 3.40 -> 197.4 mm, vias 2 -> 3
- net QTX1_P: track 4.15 -> 194.2 mm
- net PSU_DE: track 6.05 -> 195.7 mm, vias 3 -> 2
- net QRX2_P: track 3.15 -> 192.5 mm
- net QTX3_P: track 3.40 -> 192.5 mm
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Other:
- board size 240 x 190 mm -> 320 x 260 mm
