File: hardware/tr_module/SENTINEL_TRM.kicad_pcb (KiCad board)
At the start: 4 copper layers, 230 x 130 mm, 144 parts, among them J1 TX_IN, J2 RX_OUT, J3 ANT, J4 CAL, J5 BACKPLANE, J6 50V IN, J7 SWD, Q1 GaN 10W, Q2 GaN 300W, Q3 2N7002, Q4 SUD50P10, U1 GB 20dB, U10 GB 20dB, U11 LM2776, U12 DAC7311, U13 DAC7311, U14 LM321, U15 LM321, U16 LMV331, U17 74LVC1G11, U18 INA240A1, U19 LMR16006, U20 AP2112K-3.3, U21 STM32G031K8T6, U22 THVD1450, U3 CIRC 400W, U4 -30dB, U5 SPDT, U6 DET FWD, U7 DET REV, U8 LNA, U9 BPF 420-450

Commit message: Five boards DRC-clean, BOMs, layout engine improvements
- Backplane, clock & timing, calibration network, PSU and feed board layouts now pass
  KiCad DRC with zero errors and zero unconnected items
- T/R module: 0 DRC errors, 6 connections left to route by hand
- Calibration selector redesigned as an SPDT tree (replaces the fine-pitch SP8T)
- PSU: IPC-2221 2.5 mm high-voltage clearance via KiCad custom rules
- Backplane/tile cable re-pinned (slots 1-4 left column, 5-8 right) for routability
- Grouped BOM CSV for every board (hardware/tools/export_bom.sh)
- Router: partial routing, neck-downs at fine-pitch pins, long-axis fan-out,
  NPTH obstacles, pour-net connectivity, domain-aware clearance, rip-up tuning

Co-Authored-By: Claude Opus 5.5 <noreply@anthropic.com>
Parts:
- moved H3 195.2 mm to (200.0, 146.0)
- moved L11 48.6 mm to (156.1, 87.6)
- moved U13 43.1 mm to (4.47, 95.6)
- moved C31 41.7 mm to (10.5, 95.2)
- moved C46 41.3 mm to (158.2, 110.7)
- moved D6 40.8 mm to (60.5, 103.0)
- moved C45 40.3 mm to (152.6, 110.7)
- moved U16 39.5 mm to (67.1, 103.9)
- moved R46 33.6 mm to (96.5, 109.4)
- moved C40 32.2 mm to (90.5, 109.4)
- moved U11 29.9 mm to (5.08, 102.6)
- moved C32 28.5 mm to (11.7, 101.7)
- moved C33 27.2 mm to (17.7, 101.7)
- moved R32 26.8 mm to (60.5, 109.4)
- moved C34 25.8 mm to (23.9, 101.9)
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Routing:
- net +3V3: track 24.1 -> 365.9 mm, vias 21 -> 33
- net V_REFL: track 154.7 -> 5.94 mm, vias 6 -> 2
- net DRAIN_ON: track 128.0 -> 2.19 mm, vias 5 -> 2
- net Q3_G: track 138.5 -> 14.2 mm, vias 5 -> 3
- net VG_MON: track 137.1 -> 33.5 mm, vias 7 -> 4
- net DAC_CS_DRV: track 2.71 -> 83.2 mm, vias 2 -> 3
- net DAC_DIN: track 3.83 -> 79.8 mm, vias 3 -> 4
- net FAULT_N: track 96.8 -> 22.3 mm, vias 6 -> 2
- net DAC_CS_PA: track 81.9 -> 143.5 mm, vias 4 -> 2
- net LED_A: track 7.77 -> 59.6 mm, vias 2 -> 3
- net VGD_MON: track 22.4 -> 66.9 mm, vias 3 -> 4
- net VDAC_DRV: track 54.2 -> 11.5 mm, vias 4 -> 2
- net NTC_V: track 151.1 -> 111.4 mm
- net +5V: track 438.9 -> 477.9 mm, vias 20 -> 25
- net BIAS_OK: track 55.3 -> 18.2 mm, vias 3 -> 4
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Other:
- board size 230 x 130 mm -> 230 x 152 mm

Commit message: T/R module: last five nets finished with EasyEDA Pro, all 7 boards DRC clean
- +5V, DRAIN_ON, NTC_V, FAULT_N and V_REFL routed by the EasyEDA Pro
  autorouter with every existing track locked (DRAIN_ON uses one short
  In1 run); stored in tr_module/easyeda_routes.json.
- import_easyeda.py can now replace only the nets listed in the JSON.
- T/R module: 0 DRC errors, 0 unconnected; gerbers, 3D view and copper
  preview regenerated.
- Report counts tracks/vias from the board file; README now reports
  7 of 7 layouts DRC clean.

Co-Authored-By: Claude Opus 5.5 <noreply@anthropic.com>
Routing:
- net V_REFL: track 5.94 -> 134.8 mm, vias 2 -> 5
- net DRAIN_ON: track 2.19 -> 102.9 mm
- net FAULT_N: track 22.3 -> 64.9 mm, vias 2 -> 3
- net NTC_V: track 111.4 -> 149.9 mm, vias 6 -> 3
- net +5V: track 477.9 -> 483.2 mm
